File: KiCad/BlueBuzz.kicad_pcb (KiCad board)
At the start: 2 copper layers, 19.5 x 25.2 mm, 11 parts, among them J1 Conn_01x06_Socket, J2 DE9, SW1 SW_DIP_x01, SW2 SW_DIP_x01, U1 ESP32, U2 AMS1117

Commit message: update PCB
Parts:
- added J0: DE9, Connector_Dsub:DSUB-9_Pins_EdgeMount_P2.77mm, F.Cu at (154.8, 85.8)
- added J3: Conn_01x03_Socket, Jumper:SolderJumper-3_P1.3mm_Open_Pad1.0x1.5mm_NumberLabels, B.Cu at (147.2, 64.0)
- added J4: Conn_01x02_Socket, Jumper:SolderJumper-2_P1.3mm_Open_Pad1.0x1.5mm, B.Cu at (162.8, 85.8)
- added J5: Conn_01x01_Socket, Connector_Wire:SolderWirePad_1x01_SMD_1x2mm, B.Cu at (153.8, 64.0)
- added J6: Conn_01x01_Socket, Connector_Wire:SolderWirePad_1x01_SMD_1x2mm, B.Cu at (159.0, 64.0)
- J1: value Conn_01x06_Socket -> Conn_01x01_Socket; footprint Connector_Harwin:Harwin_M20-89006xx_1x06_P2.54mm_Horizontal -> Connector_Wire:SolderWirePad_1x01_SMD_1x2mm
- J2: value DE9 -> Conn_01x01_Socket; footprint Connector_Dsub:DSUB-9_Pins_EdgeMount_P2.77mm -> Connector_Wire:SolderWirePad_1x01_SMD_1x2mm; moved to B.Cu
- moved J2 22.0 mm to (155.5, 64.0), turned to 180 degrees
- moved J1 6.09 mm to (157.2, 64.0), turned to 180 degrees
Connections:
- C1 pad 1: Net-(J1-Pin_6) -> Net-(J3-Pin_1)
- C1 pad 2: Net-(J1-Pin_5) -> Net-(J4-Pin_2)
- C2 pad 1: Net-(J1-Pin_6) -> Net-(J3-Pin_1)
- J2 pad 1: Net-(U1-IO12) -> Net-(J2-Pin_1)
- R2 pad 2: Net-(J1-Pin_6) -> Net-(J3-Pin_1)
- R3 pad 2: Net-(J1-Pin_4) -> Net-(U1-EN)
- SW1 pad 1: Net-(J1-Pin_3) -> Net-(U1-IO0)
- SW1 pad 2: Net-(J1-Pin_6) -> Net-(J3-Pin_1)
- SW2 pad 1: Net-(J1-Pin_4) -> Net-(U1-EN)
- SW2 pad 2: Net-(J1-Pin_6) -> Net-(J3-Pin_1)
- U1 pad 1: Net-(J1-Pin_6) -> Net-(J3-Pin_1)
- U1 pad 15: Net-(J1-Pin_6) -> Net-(J3-Pin_1)
- U1 pad 25: Net-(J1-Pin_3) -> Net-(U1-IO0)
- U1 pad 3: Net-(J1-Pin_4) -> Net-(U1-EN)
- U1 pad 34: Net-(J1-Pin_2) -> Net-(J2-Pin_1)
- U1 pad 38: Net-(J1-Pin_6) -> Net-(J3-Pin_1)
- U1 pad 39: Net-(J1-Pin_6) -> Net-(J3-Pin_1)
- U2 pad 3: Net-(J1-Pin_5) -> Net-(J4-Pin_2)
Routing:
- net Net-(J3-Pin_1): track 0.00 -> 81.7 mm, vias 0 -> 4
- net Net-(J1-Pin_6): track 76.9 -> 0.00 mm, vias 2 -> 0
- net Net-(J1-Pin_4): track 37.8 -> 0.00 mm, vias 6 -> 0
- net Net-(J1-Pin_5): track 34.8 -> 0.00 mm, vias 2 -> 0
- net Net-(J4-Pin_2): track 0.00 -> 33.2 mm, vias 0 -> 2
- net Net-(J1-Pin_3): track 30.9 -> 0.00 mm, vias 2 -> 0
- net Net-(U1-EN): track 0.00 -> 30.1 mm, vias 0 -> 3
- net Net-(U1-IO0): track 0.00 -> 24.7 mm, vias 0 -> 1
- net Net-(J2-Pin_1): track 0.00 -> 23.9 mm, vias 0 -> 2
- net Net-(J1-Pin_1): track 4.82 -> 21.2 mm
- net Net-(J1-Pin_2): track 7.63 -> 0.00 mm, vias 1 -> 0
- net Net-(U1-IO25): track 16.6 -> 17.4 mm
- net Net-(U1-IO26): track 15.2 -> 16.0 mm
- net Net-(U1-IO33): track 19.1 -> 19.7 mm
- net Net-(U1-IO14): track 9.50 -> 10.1 mm
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Other:
- board size 19.5 x 25.2 mm -> 20 x 32 mm
- board text added: "BuzzLink"
- board text removed: "D0"
- board text removed: "EN"
- board text removed: "P1"
- board text removed: "P2"
- board text removed: "P3"
- board text removed: "P4"
- board text removed: "P5"

Commit message: 상태표시 LED 추가. 입력 전압 3.3V 변환 로직 추가. 핀배열 변경. 사용법 변경.
Parts:
- added C3: 0.1μF, Capacitor_SMD:C_0805_2012Metric, B.Cu at (161.0, 82.5)
- C1: value 10uF -> 10μF
- C2: value 22uF -> 22μF
Routing:
- net Net-(J3-Pin_1): track 81.7 -> 82.8 mm
Changed lines of the file:
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@@
 		(tags "resistor")
 		(property "Reference" "R3"
-			(at 0 1.65 180)
+			(at -1.75 0 180)
 			(layer "B.SilkS")
+			(hide yes)
 			(effects
 				(font
@@
 			)
 		)
-		(property "Value" "10uF"
+		(property "Value" "10μF"
 			(at 0 -1.68 270)
 			(layer "B.Fab")
@@
 		(embedded_fonts no)
 	)
+	(footprint "Capacitor_SMD:C_0805_2012Metric"
+		(layer "B.Cu")
+		(at 161 82.5 90)
+		(descr "Capacitor SMD 0805 (2012 Metric), square (rectangular) end terminal, IPC-7351 nominal, (Body size source: IPC-SM-782 page 76, https://www.pcb-3d.com/wordpress/wp-content/uploads/ipc-sm-782a_amendment_1_and_2.pdf, https://docs.google.com/spreadsheets/d/1BsfQQcO9C6DZCsRaXUlFlo91Tg2WpOkGARC1WS5S8t0/edit?usp=sharing), generated with kicad-footprint-generator")
+		(tags "capacitor")
+		(property "Reference" "C3"
+			(at 0.75 -1.75 180)
+			(layer "B.SilkS")
+			(effects
+				(font
+					(size 1 1)
+					(thickness 0.15)
+				)
+				(justify mirror)
+			)
+		)
+		(property "Value" "0.1μF"
+			(at 0 -1.68 90)
+			(layer "B.Fab")
+			(effects
+				(font
+					(size 1 1)
+					(thickness 0.15)
+				)
+				(justify mirror)
+			)
+		)
+		(property "Datasheet" "~"
+			(at 0 0 90)
+			(layer "B.Fab")
+			(hide yes)
+			(effects
+				(font
+					(size 1.27 1.27)
+					(thickness 0.15)
+				)
+				(justify mirror)
+			)
+		)
+		(property "Description" "Unpolarized capacitor"
+			(at 0 0 90)
+			(layer "B.Fab")
+			(hide yes)
+			(effects
+				(font
+					(size 1.27 1.27)
+					(thickness 0.15)
+				)
+				(justify mirror)
+			)
+		)
+		(property ki_fp_filters "C_*")
+		(sheetname "/")
+		(sheetfile "BlueBuzz.kicad_sch")
+		(attr smd)
+		(fp_line
+			(start -0.261252 -0.735)
+			(end 0.261252 -0.735)
+			(stroke
+				(width 0.12)
+				(type solid)
+			)
+			(layer "B.SilkS")
+		)
+		(fp_line
+			(start -0.261252 0.735)
+			(end 0.261252 0.735)
+			(stroke
+				(width 0.12)
+				(type solid)
+			)
+			(layer "B.SilkS")
+		)
+		(fp_line
+			(start 1.7 -0.98)
+			(end -1.7 -0.98)
+			(stroke
+				(width 0.05)
+				(type solid)
+			)
+			(layer "B.CrtYd")
+		)
+		(fp_line
+			(start -1.7 -0.98)
+			(end -1.7 0.98)
+			(stroke
+				(width 0.05)
+				(type solid)
+			)
+			(layer "B.CrtYd")
+		)
+		(fp_line
+			(start 1.7 0.98)
+			(end 1.7 -0.98)
+			(stroke
+				(width 0.05)
+				(type solid)
+			)
+			(layer "B.CrtYd")
+		)
+		(fp_line
+			(start -1.7 0.98)
+			(end 1.7 0.98)
+			(stroke
+				(width 0.05)
+				(type solid)
+			)
+			(layer "B.CrtYd")
+		)
+		(fp_line
+			(start 1 -0.625)
+			(end -1 -0.625)
+			(stroke
+				(width 0.1)
+				(type solid)
+			)
+			(layer "B.Fab")
+		)
+		(fp_line
+			(start -1 -0.625)
+			(end -1 0.625)
+			(stroke
+				(width 0.1)
+				(type solid)
+			)
+			(layer "B.Fab")
+		)
+		(fp_line
+			(start 1 0.625)
+			(end 1 -0.625)
+			(stroke
+				(width 0.1)
+				(type solid)
+			)
+			(layer "B.Fab")
+		)
+		(fp_line
+			(start -1 0.625)
+			(end 1 0.625)
+			(stroke
+				(width 0.1)
+				(type solid)
+			)
+			(layer "B.Fab")
+		)
+		(fp_text user "${REFERENCE}"
+			(at 0 0 90)
+			(layer "B.Fab")
+			(effects
+				(font
+					(size 0.5 0.5)
+					(thickness 0.08)
+				)
+				(justify mirror)
+			)
+		)
+		(pad "1" smd roundrect
+			(at -0.95 0 90)
+			(size 1 1.45)
+			(layers "B.Cu" "B.Mask" "B.Paste")
+			(roundrect_rratio 0.25)
+			(net 35 "Net-(U1-EN)")
+			(pintype "passive")
+		)
+		(pad "2" smd roundrect
+			(at 0.95 0 90)
+			(size 1 1.45)
+			(layers "B.Cu" "B.Mask" "B.Paste")
+			(roundrect_rratio 0.25)
+			(net 37 "Net-(J3-Pin_1)")
+			(pintype "passive")
+		)
+		(embedded_fonts no)
+		(model "${KICAD9_3DMODEL_DIR}/Capacitor_SMD.3dshapes/C_0805_2012Metric.step"
+			(offset
+				(xyz 0 0 0)
+			)
+			(scale
+				(xyz 1 1 1)
+			)
+			(rotate
+				(xyz 0 0 0)
+			)
+		)
+	)
 	(footprint "Jumper:SolderJumper-2_P1.3mm_Open_Pad1.0x1.5mm"
 		(layer "B.Cu")
@@
 		(tags "resistor")
 		(property "Reference" "R2"
-			(at 2.5 0 180)
+			(at 2.25 0 180)
 			(layer "B.SilkS")
 			(effects
@@
 			)
 		)
-		(property "Value" "22uF"
+		(property "Value" "22μF"
 			(at 0 -1.68 270)
 			(layer "B.Fab")
@@
 	(segment
 		(start 163.25 83.4125)
-		(end 159.9125 83.4125)
+		(end 161 83.4125)
+		(width 0.2)
+		(layer "B.Cu")
+		(net 35)
+	)
+	(segment
+		(start 161 83.45)
+		(end 161 83.4125)
 		(width 0.2)
 		(layer "B.Cu")
@@
 	)
 	(segment
+		(start 161 83.4125)
+		(end 159.9125 83.4125)
+		(width 0.2)
+		(layer "B.Cu")
+		(net 35)
+	)
+	(segment
 		(start 154.125 77.125)
 		(end 154 77)
@@
 	)
 	(segment
+		(start 161 81.55)
+		(end 161 80.6625)
+		(width 0.2)
+		(layer "B.Cu")
+		(net 37)
+	)
+	(segment
 		(start 158.75 80.45)
 		(end 158.75 82.01)
@@
 		(width 0.2)
 		(layer "B.Cu")
+		(net 37)
+	)
+	(segment
+		(start 161 80.6625)
+		(end 161.2125 80.45)
+		(width 0.2)
+		(layer "B.Cu")
